Commit message: Milestone 1 done

File: body1.urdf (robot description, URDF)
Before this commit: robot robot, 9 links, 8 joints
Joints:
- joint BackLeg_LowerBackLeg: axis 3 0 2 -> 1 0 0
- joint FrontLeg_LowerFrontLeg: axis 3 0 2 -> 1 0 0
- joint LeftLeg_LowerLeftLeg: axis 3 0 3 -> 1 0 1
- joint RightLeg_LowerRightLeg: axis 3 0 3 -> 1 0 1
- joint Torso_BackLeg: axis 3 0 2 -> 1 0 0
- joint Torso_FrontLeg: axis 3 0 2 -> 1 0 0
- joint Torso_LeftLeg: axis 3 0 3 -> 1 0 1
- joint Torso_RightLeg: axis 3 0 3 -> 1 0 1

Commit message: Finsihed last one

File: body1.urdf (robot description, URDF)
Before this commit: robot robot, 13 links, 12 joints
Links:
- removed link BackLeg2
- removed link FrontLeg2
- removed link LowerBackLeg2
- removed link LowerFrontLeg2
Joints:
- removed joint BackLeg2_LowerBackLeg2
- removed joint FrontLeg2_LowerFrontLeg
- removed joint Torso_BackLeg2
- removed joint Torso_FrontLeg2
